File: PCB/Base Circuit/MCU & Communication.kicad_sch (KiCad schematic)
At the start: 9 parts, among them J1 Raspberry_Pi_4, U1 ESP32-DEVKITC-32D

Commit message: PCB Updated
Parts:
- removed MCP2515_CAN_MODULE: Conn_01x09, symbol Connector_Generic:Conn_01x09
- added JMCP2515_CAN_MODULE: Conn_01x07, symbol Connector_Generic:Conn_01x07
- added MCP2515_CAN_MODULE_T-BLOCK: Conn_01x02, symbol Connector_Generic:Conn_01x02
Connections:
- net DIR_MFL is gone; now on net A3_VD: U1.J3-13 (IO4)
- net DIR_MFL_B is gone; now on net B3_VD: U1.J3-12 (IO16)
- net PWM_MFL is gone; now on net B4_VD: U1.J3-10 (IO5)
- net 3.3V: now also JMCP2515_CAN_MODULE.1 (Pin_1)
- net 5V: no longer J1.2 (5V), J1.4 (5V)
- net A2_VD: now also U1.J2-3 (SENSOR_VP); no longer U1.J3-11 (IO17)
- net A3_VD: no longer U1.J3-16 (IO15)
- net A4_VD: now also U1.J3-11 (IO17); no longer U1.J2-3 (SENSOR_VP)
- net B2_VD: now also U1.J2-4 (SENSOR_VN); no longer U1.J3-15 (IO2)
- net B3_VD: no longer U1.J3-14 (IO0)
- net B4_VD: no longer U1.J2-4 (SENSOR_VN)
- net CANH: now also MCP2515_CAN_MODULE_T-BLOCK.1 (Pin_1)
- net CANL: now also MCP2515_CAN_MODULE_T-BLOCK.2 (Pin_2)
- net CS: now also JMCP2515_CAN_MODULE.3 (Pin_3)
- net GND: now also JMCP2515_CAN_MODULE.2 (Pin_2)
- net INT: now also JMCP2515_CAN_MODULE.7 (Pin_7)
- net SCK: now also JMCP2515_CAN_MODULE.6 (Pin_6)
- net SI: now also JMCP2515_CAN_MODULE.5 (Pin_5)
- net SO: now also JMCP2515_CAN_MODULE.4 (Pin_4)
- net DIR_MBL renamed MFR_IN1
- net DIR_MBL_B renamed MFR_IN2
- net DIR_MBR renamed MBR_IN2
- net DIR_MBR_B renamed MBL_IN1
- net DIR_MFR renamed MFL_IN2
- net DIR_MFR_B: no longer names the net of U1.J3-2 (IO23)
- net PWM_MBL renamed MBL_IN2
- net PWM_MBR renamed MBR_IN1
- net PWM_MFR renamed MFL_IN1
- new net 5V_RASPBEERY: J1.2 (5V), J1.4 (5V)
