File: PCB/PCB Design KICAD/MCU & Communication.kicad_sch (KiCad schematic)
At the start: 16 parts, among them J1 Raspberry_Pi_4, J2 Conn_01x02_Pin, J3 Conn_01x02_Pin, J4 Conn_01x02_Pin, J5 Conn_01x02_Pin, U1 ESP32-DEVKITC-32D

Commit message: FINAL SCHEMATIC
Parts:
- CAN_BUS1: renamed from CAN_BUS; footprint (none) -> TerminalBlock:TerminalBlock_MaiXu_MX126-5.0-03P_1x03_P5.00mm
- J2: renamed from J3; footprint (none) -> Connector_PinHeader_2.54mm:PinHeader_1x02_P2.54mm_Vertical
- J3: renamed from J4; footprint (none) -> Connector_PinHeader_2.54mm:PinHeader_1x02_P2.54mm_Vertical
- J4: renamed from J2; footprint (none) -> Connector_PinHeader_2.54mm:PinHeader_1x02_P2.54mm_Vertical
- J5: footprint (none) -> Connector_PinHeader_2.54mm:PinHeader_1x02_P2.54mm_Vertical
- JMCP2515_CAN_MODULE1: renamed from JMCP2515_CAN_MODULE; footprint (none) -> Connector_PinHeader_2.54mm:PinHeader_1x07_P2.54mm_Vertical
- Jumper_Shunt1: renamed from Jumper_Shunt; footprint (none) -> Connector_PinHeader_2.54mm:PinHeader_1x03_P2.54mm_Vertical
- Jumper_Shunt2: renamed from Jumper_Shunt1; footprint (none) -> Connector_PinHeader_2.54mm:PinHeader_1x03_P2.54mm_Vertical
- MCP2515_CAN_MODULE_T-BLOCK1: renamed from MCP2515_CAN_MODULE_T-BLOCK; footprint (none) -> Connector_PinHeader_2.54mm:PinHeader_1x02_P2.54mm_Vertical
- RASPBERRY_PI1: renamed from J1; footprint (none) -> Connector_IDC:IDC-Header_2x20_P2.54mm_Vertical
- RS485_ESP1: renamed from RS485_ESP; footprint (none) -> Library:MODULE_MAX485_MODULE_5V_LOGIC_TLL_TO_RS-485_CONVERTER
- RS485_RASP1: renamed from RS485_RASP; footprint (none) -> Library:MODULE_MAX485_MODULE_5V_LOGIC_TLL_TO_RS-485_CONVERTER
- RS_BUS1: renamed from RS_BUS; footprint (none) -> TerminalBlock:TerminalBlock_MaiXu_MX126-5.0-03P_1x03_P5.00mm
- SN65HVD230_MODULE1: renamed from SN65HVD230_MODULE; footprint (none) -> Connector_PinSocket_2.54mm:PinSocket_1x06_P2.54mm_Vertical
- Termination_Resistor1: renamed from Termination_Resistor; footprint (none) -> Resistor_THT:R_Axial_DIN0207_L6.3mm_D2.5mm_P7.62mm_Horizontal
- U2: renamed from U1; footprint ESP32-DEVKITC-32D:MODULE_ESP32-DEVKITC-32D -> Library:MODULE_ESP32-DEVKITC-32D
Other:
- moved on the sheet: MCP2515_CAN_MODULE_T-BLOCK1

Commit message: Final schematic updated
Parts:
- RS485_ESP1, RS485_RASP1: footprint Library:MODULE_MAX485_MODULE_5V_LOGIC_TLL_TO_RS-485_CONVERTER -> Library:ECO-MAX485-TTL-TO-RS-485-MODULE
Changed lines of the file:
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@@
 			)
 		)
-		(property "Footprint" "Library:MODULE_MAX485_MODULE_5V_LOGIC_TLL_TO_RS-485_CONVERTER"
+		(property "Footprint" "Library:ECO-MAX485-TTL-TO-RS-485-MODULE"
 			(at 237.49 107.95 0)
 			(effects
@@
 			)
 		)
-		(property "Footprint" "Library:MODULE_MAX485_MODULE_5V_LOGIC_TLL_TO_RS-485_CONVERTER"
+		(property "Footprint" "Library:ECO-MAX485-TTL-TO-RS-485-MODULE"
 			(at 237.49 147.32 0)
 			(effects
