File: PCB/PCB Design KICAD/Power & Regulation.kicad_sch (KiCad schematic)
At the start: 25 parts, among them SW1_ESTOP SW_SPST

Commit message: FINAL SCHEMATIC
Parts:
- removed Main_Buck, Raspberry_Buck: DCBuck, PrntrBoardV2:Buck2217, symbol BuckConverter:DCBuck
- added BUCK_MAIN1: MP1584EN DC-DC Buck Converter, Library:EBOOT MINI MP1584EN DC-DC BUCK CONVERTER ADJUSTABLE POWER STEP DOWN MODULE 24V TO 12V 9V 5V 3V, 6 PACK, symbol New_Library:eBoot Mini MP1584EN DC-DC Buck Converter Adjustable Power Step Down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
- added BUCK_RASP1: XL4015 DC-DC STEP DOWN MODULE, Library:XL4015 DC-DC STEP DOWN MODULE, symbol New_Library:XL4015 DC-DC STEP DOWN MODULE
- BMS1: renamed from Charger; footprint (none) -> TerminalBlock:TerminalBlock_MaiXu_MX126-5.0-02P_1x02_P5.00mm
- Bridge_Rec.1: renamed from Bridge_Rec.; footprint (none) -> Library:DIO-BG-TH_KBPC3510
- C1, C4: renamed from C?; footprint PrntrBoardV2:C_0603_1608Metric -> Capacitor_THT:CP_Radial_D5.0mm_P2.50mm
- C2, C3: renamed from C?; footprint PrntrBoardV2:C_0603_1608Metric -> Capacitor_THT:C_Disc_D3.8mm_W2.6mm_P2.50mm
- C5: renamed from C1; footprint (none) -> Capacitor_THT:CP_Radial_D10.0mm_P5.00mm
- C6: renamed from C2; footprint (none) -> Capacitor_THT:C_Disc_D3.8mm_W2.6mm_P2.50mm
- Charger1: renamed from BMS; footprint (none) -> TerminalBlock:TerminalBlock_MaiXu_MX126-5.0-02P_1x02_P5.00mm
- D1: renamed from D2; footprint (none) -> LED_THT:LED_D3.0mm
- D2: renamed from D1; footprint (none) -> LED_THT:LED_D3.0mm
- D3: footprint (none) -> LED_THT:LED_D3.0mm
- F1_MAIN1: renamed from F1_MAIN; footprint (none) -> Connector_PinHeader_2.54mm:PinHeader_1x01_P2.54mm_Horizontal
- R1: renamed from R3; footprint (none) -> Resistor_THT:R_Axial_DIN0207_L6.3mm_D2.5mm_P7.62mm_Horizontal
- R2: footprint (none) -> Resistor_THT:R_Axial_DIN0207_L6.3mm_D2.5mm_P7.62mm_Horizontal
- R3: renamed from R1; footprint (none) -> Resistor_THT:R_Axial_DIN0207_L6.3mm_D2.5mm_P7.62mm_Horizontal
- SW1_ESTOP1: renamed from SW1_ESTOP; footprint (none) -> TerminalBlock:TerminalBlock_MaiXu_MX126-5.0-02P_1x02_P5.00mm
- TP1: renamed from TP?; footprint (none) -> TestPoint:TestPoint_THTPad_1.0x1.0mm_Drill0.5mm
- TP2: footprint (none) -> TestPoint:TestPoint_THTPad_1.0x1.0mm_Drill0.5mm
- TP3: renamed from TP1; footprint (none) -> TestPoint:TestPoint_THTPad_1.0x1.0mm_Drill0.5mm
- TP4: renamed from TP3; footprint (none) -> TestPoint:TestPoint_THTPad_1.0x1.0mm_Drill0.5mm
- gave numbers to parts that had none: 1
- renumbered D1_TVS to D1_TVS1
Connections:
- net 12V: now also BUCK_MAIN1.2 ((+)), BUCK_RASP1.1 (+)
- net 5V: now also BUCK_MAIN1.4 ((+))
- net 5V_RASPBEERY: now also BUCK_RASP1.2 (+)
- net GND: now also BUCK_MAIN1.1 ((-)), BUCK_MAIN1.3 ((-)), BUCK_RASP1.3 (-), BUCK_RASP1.4 (-)
Other:
- moved on the sheet: TP1, TP4

Commit message: Final schematic updated
Parts:
- BMS1: footprint TerminalBlock:TerminalBlock_MaiXu_MX126-5.0-02P_1x02_P5.00mm -> Connector_BarrelJack:BarrelJack_GCT_DCJ200-10-A_Horizontal
Changed lines of the file:
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@@
 			)
 		)
-		(property "Footprint" "TerminalBlock:TerminalBlock_MaiXu_MX126-5.0-02P_1x02_P5.00mm"
+		(property "Footprint" "Connector_BarrelJack:BarrelJack_GCT_DCJ200-10-A_Horizontal"
 			(at 208.28 68.326 0)
 			(effects
